Commit message: updating

File: cameras/bumblebee/bumblebee2.urdf.xacro (robot description, xacro)
@@ -15,5 +15,5 @@
     <link name="${frame_prefix}mount_link">
       <visual>
-        <origin xyz="0 0 0" rpy="3.14159 0 0"/>
+        <origin xyz="0 0 0" rpy="0 0 0"/>
         <geometry>
           <mesh filename="package://lcsr_camera_models/cameras/bumblebee/bumblebee2.dae"/>
@@ -21,5 +21,5 @@
       </visual>
       <collision>
-        <origin xyz="0 0 0" rpy="3.14159 0 0"/>
+        <origin xyz="0 0 0" rpy="0 0 0"/>
         <geometry>
           <mesh filename="package://lcsr_camera_models/cameras/bumblebee/bumblebee2.dae"/>

Commit message: changing frame convention to conform to standard ros camera calibration: optical frame corresponds to the left camera, instead of the location between the cameras

File: cameras/bumblebee/bumblebee2.urdf.xacro (robot description, xacro)
@@ -7,5 +7,6 @@
   <xacro:property name="b2ly" value="0.036"/>
   <xacro:property name="b2lz" value="0.0474"/>
-  <xacro:macro name="bumblebee2" params="parent_link xyz rpy ns frame_prefix high_res hfov">
+  <xacro:macro name="bumblebee2"
+    params="parent_link xyz rpy optical_parent_link optical_xyz optical_rpy ns frame_prefix high_res hfov">
     <joint name="bumblebee2_mount_joint" type="fixed">
       <parent link="${parent_link}"/>
@@ -35,15 +36,15 @@
     </link>
     <joint name="${frame_prefix}optical_joint" type="fixed">
-      <parent link="${frame_prefix}mount_link"/>
+      <parent link="${optical_parent_link}"/>
       <child link="${frame_prefix}optical_frame"/>
-      <origin xyz="0 0 0" rpy="0 0 0"/>
+      <origin xyz="${optical_xyz}" rpy="${optical_rpy}"/>
     </joint>
     <link name="${frame_prefix}optical_frame">
       <inertial>
-        <mass value="1E-6" />
+        <mass value="1E-5" />
         <inertia
-          ixx="1E-6" ixy="0" ixz="0"
-          iyy="1E-6" iyz="0"
-          izz="1E-6" />
+          ixx="1E-10" ixy="0" ixz="0"
+          iyy="1E-10" iyz="0"
+          izz="1E-10" />
       </inertial>
     </link>
@@ -58,5 +59,7 @@
         width="1024"
         height="768"
-        format="R8G8B8"/>
+        format="R8G8B8"
+        near="0.05"
+        far="300"/>
     </xacro:if>
     <xacro:unless value="${high_res}">
@@ -76,9 +79,12 @@
   </xacro:macro>
   <!-- A bumblebee with a 97-degre HFOV lens -->
-  <xacro:macro name="bumblebee2_97" params="parent_link xyz rpy ns frame_prefix high_res">
+  <xacro:macro name="bumblebee2_97" params="parent_link xyz rpy optical_parent_link optical_xyz optical_rpy ns frame_prefix high_res">
     <xacro:bumblebee2
       parent_link="${parent_link}"
       xyz="${xyz}"
       rpy="${rpy}"
+      optical_parent_link="${optical_parent_link}"
+      optical_xyz="${optical_xyz}"
+      optical_rpy="${optical_rpy}"
       ns="${ns}"
       frame_prefix="${frame_prefix}"
@@ -87,9 +93,12 @@
   </xacro:macro>
   <!-- A bumblebee with a 66-degre HFOV lens -->
-  <xacro:macro name="bumblebee2_66" params="parent_link xyz rpy ns frame_prefix high_res">
+  <xacro:macro name="bumblebee2_66" params="parent_link xyz rpy optical_parent_link optical_xyz optical_rpy ns frame_prefix high_res">
     <xacro:bumblebee2
       parent_link="${parent_link}"
       xyz="${xyz}"
       rpy="${rpy}"
+      optical_parent_link="${optical_parent_link}"
+      optical_xyz="${optical_xyz}"
+      optical_rpy="${optical_rpy}"
       ns="${ns}"
       frame_prefix="${frame_prefix}"
@@ -98,9 +107,12 @@
   </xacro:macro>
   <!-- A bumblebee with a 43-degre HFOV lens -->
-  <xacro:macro name="bumblebee2_43" params="parent_link xyz rpy ns frame_prefix high_res">
+  <xacro:macro name="bumblebee2_43" params="parent_link xyz rpy optical_parent_link optical_xyz optical_rpy ns frame_prefix high_res">
     <xacro:bumblebee2
       parent_link="${parent_link}"
       xyz="${xyz}"
       rpy="${rpy}"
+      optical_parent_link="${optical_parent_link}"
+      optical_xyz="${optical_xyz}"
+      optical_rpy="${optical_rpy}"
       ns="${ns}"
       frame_prefix="${frame_prefix}"

File: stereo_camera.urdf.xacro (robot description, xacro)
@@ -7,5 +7,5 @@
         <update_rate>${update_rate}</update_rate>
         <camera name="left">
-          <pose>${baseline / 2.0} 0 0 0 1.5707 1.5707</pose>
+          <pose>0 0 0 0 -1.5707 1.5707</pose>
           <horizontal_fov>${hfov}</horizontal_fov>
           <image>
@@ -25,5 +25,5 @@
         </camera>
         <camera name="right">
-          <pose>${-baseline / 2.0} 0 0 0 1.5707 1.5707</pose>
+          <pose>${baseline} 0 0 0 -1.5707 1.5707</pose>
           <horizontal_fov>${hfov}</horizontal_fov>
           <image>

File: test.urdf.xacro (robot description, xacro)
@@ -6,5 +6,8 @@
     parent_link="world"
     xyz="0 0 1.0"
-    rpy="1.5707 0 0"
+    rpy="1.5707 3.1416 0"
+    optical_parent_link="world"
+    optical_xyz="0.06 0 1.0"
+    optical_rpy="1.5707 3.1416 0"
     ns="bumblebee"
     frame_prefix="bumblebee_"
